File: Duo.kicad_sch (KiCad schematic)
At the start: 19 parts, among them U1 STM32H573RITx, U2 STM32H573RITx, Y1 Crystal

Commit message: Update
Parts:
- added C13, C14: 30pF, Capacitor_SMD:C_0402_1005Metric, symbol Device:C
- added C15, C16, C18, C20: 100nF, Capacitor_SMD:C_0402_1005Metric, symbol Device:C
- added C17, C19, C21: 10uF, Capacitor_SMD:C_0603_1608Metric, symbol Device:C
- added D2: CLMVC-FKA-CL1D1L71BB7C3C3, DuoFootprints:LED_CLMVC-FKA-CL1D1L71BB7C3C3, symbol CLMVC-FKA-CL1D1L71BB7C3C3:CLMVC-FKA-CL1D1L71BB7C3C3
- added D3: 1N5819HW-7-F, DuoFootprints:SOD3715X145N, symbol MyParts:1N5819HW-7-F
- added D4: PWR, LED_SMD:LED_0603_1608Metric, symbol Device:LED
- added J1: UJ20-C-H-G-SMT-P16-TR, DuoFootprints:SAMESKY_UJ20-C-H-G-SMT-P16-TR, symbol UJ20-C-H-G-SMT-P16-TR:UJ20-C-H-G-SMT-P16-TR
- added J2, J4: ~, DuoFootprints:PinHeader-Castellated-12, symbol PinHeaders:PinHeader_12
- added J3: ~, DuoFootprints:PinHeader-Castellated-8, symbol PinHeaders:PinHeader_8
- added J5: DEBUG, Connector_PinHeader_2.54mm:PinHeader_1x06_P2.54mm_Vertical, symbol Connector_Generic:Conn_01x06
- added Q1, Q2, Q3: DMG1012UW-7, Package_TO_SOT_SMD:SOT-323_SC-70, symbol Transistor_FET:DMG1012T
- added R10, R9: 5k1, Resistor_SMD:R_0402_1005Metric, symbol Device:R
- added R11, R13, R4: 221R, Resistor_SMD:R_0402_1005Metric, symbol Device:R
- added R12, R14, R15, R5: 10k, Resistor_SMD:R_0402_1005Metric, symbol Device:R
- added R6: 1k4, Resistor_SMD:R_0402_1005Metric, symbol Device:R
- added R7: 1k1, Resistor_SMD:R_0402_1005Metric, symbol Device:R
- added R8: 160R, Resistor_SMD:R_0402_1005Metric, symbol Device:R
- added SW1, SW2: PTS810_SJM_250_SMTR_LFS, DuoFootprints:SW_PTS810_SJM_250_SMTR_LFS, symbol PTS810_SJM_250_SMTR_LFS:PTS810_SJM_250_SMTR_LFS
- added U2: USBLC6-2SC6, Package_TO_SOT_SMD:SOT-23-6, symbol Power_Protection:USBLC6-2SC6
- added U3: LD1117S33TR_SOT223, Package_TO_SOT_SMD:SOT-223-3_TabPin2, symbol Regulator_Linear:LD1117S33TR_SOT223
- added Y2: ECS-80-18-23B-JTN-TR, DuoFootprints:XTAL_ECS-80-18-23B-JTN-TR, symbol ECS-80-18-23B-JTN-TR:ECS-80-18-23B-JTN-TR
- renumbered C21 to C1, C28 to C10, C29 to C11, C30 to C12, C3 to C2, C22 to C3, C23 to C4, C16 to C5, C24 to C6, C25 to C7, C26 to C8, C27 to C9, R4 to R2, R7 to R3, U2 to U1
Connections:
- net +3V3: now also C15.1, C21.1, D2.1, J4.11, J5.1 (Pin_1), R15.2, SW1.1, SW1.2, U3.2 (VO)
- net BOOT0: now also C16.1, SW1.3, SW1.4
- net GND: now also C13.2, C14.2, C15.2, C16.2, C17.2, C18.2, C19.2, C20.2, C21.2, D4.1 (K), J1.A12_B1 (GND), J1.A1_B12 (GND), J4.10, J5.6 (Pin_6), Q1.2 (S), Q2.2 (S), Q3.2 (S), R10.2, R12.1, R14.1, R5.1, R9.2, SW2.1, SW2.2, U2.2 (GND), U3.1 (GND), Y2.2, Y2.4
- net NRST: now also C18.1, J5.5 (Pin_5), SW2.3, SW2.4
- net PC2: now reaches U1.10 (PC2)
- net PC2: now also J2.3
- net PC3: now reaches U1.11 (PC3)
- net PC3: now also J2.4
- net PA0: now reaches U1.14 (PA0)
- net PA0: now also J2.6
- net PA1: now reaches U1.15 (PA1)
- net PA1: now also J2.7
- net PA2: now reaches U1.16 (PA2)
- net PA2: now also J2.8
- net PA3: now reaches U1.17 (PA3)
- net PA3: now also J2.9
- net PA4: now reaches U1.20 (PA4)
- net PA4: now also J2.10
- net PA5: now reaches U1.21 (PA5)
- net PA5: now also J2.11
- net PA6: now reaches U1.22 (PA6)
- net PA6: now also J2.12
- net PA7: now reaches U1.23 (PA7)
- net PA7: now also J3.1
- net PC4: now reaches U1.24 (PC4)
- net PC4: now also J2.5
- net PB0: now reaches U1.26 (PB0)
- net PB0: now also J3.2
- net PB10: now reaches U1.29 (PB10)
- net PB10: now also J3.3
- net PB12: now reaches U1.33 (PB12)
- net PB12: now also J3.4
- net PB13: now reaches U1.34 (PB13)
- net PB13: now also J3.5
- net PB14: now reaches U1.35 (PB14)
- net PB14: now also J3.6
- net PB15: now reaches U1.36 (PB15)
- net PB15: now also J3.7
- net RGB_RED: now reaches U1.37 (PC6)
- net RGB_RED: now also R13.2
- net RGB_GREEN: now reaches U1.38 (PC7)
- net RGB_GREEN: now also R11.2
- net RGB_BLUE: now reaches U1.39 (PC8)
- net RGB_BLUE: now also R4.2
- net PC9: now reaches U1.40 (PC9)
- net PA8: now reaches U1.41 (PA8)
- net PA8: now also J3.8
- net PA9: now reaches U1.42 (PA9)
- net PA9: now also J4.1
- net PA10: now reaches U1.43 (PA10)
- net PA10: now also J4.2
- net D-: now reaches U1.44 (PA11)
- net D-: now also U2.6 (I/O1)
- net D+: now reaches U1.45 (PA12)
- net D+: now also U2.4 (I/O2)
- net SWDIO: now reaches U1.46 (PA13)
- net SWDIO: now also J5.2 (Pin_2)
- net SWCLK: now reaches U1.49 (PA14)
- net SWCLK: now also J5.3 (Pin_3)
- net at U1.5 (PH0-OSC_IN): now also C14.1, Y2.3
- net PC10: now reaches U1.51 (PC10)
- net PC10: now also J4.3
- net PC11: now reaches U1.52 (PC11)
- net PC11: now also J4.4
- net PC12: now reaches U1.53 (PC12)
- net PC12: now also J4.5
- net PD2: now reaches U1.54 (PD2)
- net PD2: now also J4.6
- net SWO: now reaches U1.55 (PB3)
- net SWO: now also J5.4 (Pin_4)
- net PB6: now reaches U1.58 (PB6)
- net PB6: now also J4.7
- net PB7: now reaches U1.59 (PB7)
- net PB7: now also J4.8
- net at U1.6 (PH1-OSC_OUT): now also C13.1, Y2.1
- net PB8: now reaches U1.61 (PB8)
- net PB8: now also J4.9
- net PC0: now reaches U1.8 (PC0)
- net PC0: now also J2.1
- net PC1: now reaches U1.9 (PC1)
- net PC1: now also J2.2
- new net: D4.2 (A), R15.1
- new net: J1.A7 (DN1), J1.B7 (DN2), U2.1 (I/O1)
- new net: J1.A6 (DP1), J1.B6 (DP2), U2.3 (I/O2)
- new net: Q1.1 (G), R4.1, R5.2
- new net: Q3.1 (G), R13.1, R14.2
- new net: J1.A5 (CC1), R10.1
- new net: J1.B5 (CC2), R9.1
- new net: J1.SH1 (SHIELD), J1.SH2 (SHIELD), J1.SH3 (SHIELD), J1.SH4 (SHIELD)
- new net: D2.4, R6.1
- new net: Q3.3 (D), R6.2
- new net: Q2.1 (G), R11.1, R12.2
- new net: D2.3, R7.1
- new net: Q2.3 (D), R7.2
- new net: Q1.3 (D), R8.2
- new net: D2.2, R8.1
- new net +5V: C17.1, C19.1, C20.1, D3.C, J4.12, U2.5 (VBUS), U3.3 (VI)
- new net VBUS: D3.A, J1.A4_B9 (VBUS), J1.A9_B4 (VBUS)
- no-connect marks 0 -> 3
Other:
- note added: "BOOT/RST"
- note added: "RGB LED"
- note added: "STM32H5"
- note added: "USB-C"
- note added: "Voltage Regulator"
- moved on the sheet: C1, C10, C11, C12, C2, C3, C4, C5, C6, C7, C8, C9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
